Commit message: 5 dof and 2 dof options are added

File: src/the_turk_core/urdf/the_turk.urdf (robot description, URDF)
Before this commit: robot the_turk, 7 links, 6 joints
Links:
- link base_link: mass None -> 4.8; geometry collision cylinder length=0.24 radius=0.24; visual box size=0.018 0.12 0.012
- link gripper_base: mass None -> 0.55; geometry collision box size=0.16 0.12 0.11; visual box size=0.095 0.08 0.010
- link left_finger: mass None -> 0.16; geometry collision box size=0.045 0.045 0.20; visual box size=0.045 0.045 0.05
- link link1: mass None -> 3.2; geometry collision box size=0.16 0.17 0.58; visual box size=0.008 0.065 0.24
- link link2: mass None -> 2.1; geometry collision box size=0.14 0.15 0.48; visual box size=0.006 0.055 0.17
- link right_finger: mass None -> 0.16; geometry collision box size=0.045 0.045 0.20; visual box size=0.045 0.045 0.05
- link wrist_link: mass None -> 0.65; geometry collision cylinder length=0.18 radius=0.08; visual cylinder length=0.012 radius=0.075
